File: phocuser.kicad_pcb (KiCad board)
At the start: 4 copper layers, 35 x 40 mm, 55 parts, among them J1 Conn_01x04_Male, J2 Conn_ARM_JTAG_SWD_10, J3 Conn_01x02_Male, J4 DX07S016JA1R1500, J5 Accessory 0, J6 Accessory 1, J7 USB, J8 Accessory 2, U1 HolyIot-18010, U2 TMC2130-LA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

Commit message: Design sent to OshPark 9/14/2022
Parts:
- added C19: 470nF, Capacitor_SMD:C_0402_1005Metric, F.Cu at (196.4, 80.1)
- added D3: LED, LED_SMD:LED_0603_1608Metric, F.Cu at (177.4, 79.7)
- added D4: LED, LED_SMD:LED_0603_1608Metric, F.Cu at (179.0, 79.7)
- added R15: 470, Resistor_SMD:R_0402_1005Metric, F.Cu at (181.2, 82.8)
- added R16: 470, Resistor_SMD:R_0402_1005Metric, F.Cu at (179.4, 81.8)
- added R20: 47k, Resistor_SMD:R_0402_1005Metric, F.Cu at (197.4, 80.1)
- added R21: 10k, Resistor_SMD:R_0402_1005Metric, F.Cu at (196.4, 78.2)
Connections:
- U1 pad 15: unconnected-(U1-Pad15) -> Net-(U1-Pad15)
- U1 pad 16: unconnected-(U1-Pad16) -> Net-(U1-Pad16)
- U1 pad 2: ACC0_A -> unconnected-(U1-Pad2)
- U1 pad 3: ACC0_B -> /Vmeas
- U1 pad 35: unconnected-(U1-Pad35) -> ACC0_A
- U1 pad 36: unconnected-(U1-Pad36) -> ACC0_B
Routing:
- net /Vmeas: track 0.00 -> 23.4 mm, vias 0 -> 1
- net ACC0_B: track 8.66 -> 22.8 mm, vias 0 -> 1
- net ACC0_A: track 6.90 -> 20.4 mm, vias 0 -> 1
- net Net-(D3-Pad2): track 0.00 -> 4.96 mm
- net GND: track 39.8 -> 44.4 mm, vias 27 -> 30
- net Net-(U1-Pad15): track 0.00 -> 2.12 mm, vias 0 -> 1
- net Net-(U1-Pad16): track 0.00 -> 1.81 mm, vias 0 -> 1
- net Net-(D4-Pad2): track 0.00 -> 1.35 mm
- net +12V: track 14.2 -> 15.1 mm, vias 5 -> 6
