File: phocuser.kicad_sch (KiCad schematic)
At the start: 54 parts, among them U3 FT231XQ

Commit message: edits
Parts:
- added J8: Accessory 2, Connector_JST:JST_PH_B4B-PH-K_1x04_P2.00mm_Vertical, symbol Connector:Conn_01x04_Male
- J7: value (none) -> USB
Connections:
- net ACC0_A: now also U1.2 (P1.11); no longer U1.6 (P0.03)
- net ACC0_B: now also U1.3 (P1.10); no longer U1.7 (P0.02)
- net ACC1_A: now also U1.6 (P0.03); no longer U1.10 (P0.30)
- net ACC1_B: now also U1.5 (P1.15); no longer U1.9 (P0.29)
- net GND: now also J8.4 (Pin_4)
- net MOSI: now also U1.10 (P0.30); no longer U1.5 (P1.15)
- net SCLK: now also U1.9 (P0.29); no longer U1.4 (P1.13)
- net THERM0: now also U1.4 (P1.13); no longer U1.8 (P0.28)
- net TMCCLK: now also U1.7 (P0.02); no longer U1.2 (P1.11)
- net ~{CS1}: now also U1.8 (P0.28); no longer U1.3 (P1.10)
- net ACC2_C: now reaches U1.28 (P1.03)
- net ACC2_C: now also J8.3 (Pin_3)
- net ACC2_B: now reaches U1.29 (P1.01)
- net ACC2_B: now also J8.2 (Pin_2)
- net ACC2_A: now reaches U1.30 (P1.02)
- net ACC2_A: now also J8.1 (Pin_1)
- net at U2.13 (OB1): now also J1.2 (Pin_2); no longer J1.1 (Pin_1)
- net at U2.15 (OB2): now also J1.1 (Pin_1); no longer J1.2 (Pin_2)
- net at U2.32 (OA2): now also J1.4 (Pin_4); no longer J1.3 (Pin_3)
- net at U2.34 (OA1): now also J1.3 (Pin_3); no longer J1.4 (Pin_4)

Commit message: Design sent to OshPark 9/14/2022
Parts:
- added C19: 470nF, Capacitor_SMD:C_0402_1005Metric, symbol Device:C
- added D3, D4: LED, LED_SMD:LED_0603_1608Metric, symbol Device:LED
- added R15, R16: 470, Resistor_SMD:R_0402_1005Metric, symbol Device:R_US
- added R20: 47k, Resistor_SMD:R_0402_1005Metric, symbol Device:R_US
- added R21: 10k, Resistor_SMD:R_0402_1005Metric, symbol Device:R_US
- C1: value (none) -> 470nF; footprint (none) -> Capacitor_SMD:C_0402_1005Metric
- C10, C14, C15, C16, C17, C18, C4, C5, C6, C7, C9: value (none) -> 100nf; footprint (none) -> Capacitor_SMD:C_0402_1005Metric
- C11: value (none) -> 10nf; footprint (none) -> Capacitor_SMD:C_0402_1005Metric
- C12, C13: value (none) -> 27pf; footprint (none) -> Capacitor_SMD:C_0402_1005Metric
- C2: value (none) -> 4.7U; footprint (none) -> Capacitor_SMD:C_0805_2012Metric
- C3: value (none) -> 22nf; footprint (none) -> Capacitor_SMD:C_0402_1005Metric
- C8: value (none) -> 10u; footprint (none) -> Capacitor_SMD:C_0805_2012Metric
- D1: value (none) -> LED; footprint (none) -> LED_SMD:LED_0603_1608Metric
- FB1: value (none) -> Ferrite_Bead; footprint (none) -> Inductor_SMD:L_0402_1005Metric
- J1: value (none) -> Conn_01x04_Male; footprint (none) -> Connector_JST:JST_XH_B4B-XH-A_1x04_P2.50mm_Vertical
- J2: value (none) -> Conn_ARM_JTAG_SWD_10; footprint (none) -> Connector_PinHeader_1.27mm:PinHeader_2x05_P1.27mm_Vertical_SMD
- J3: value (none) -> Conn_01x02_Male; footprint (none) -> Connector_JST:JST_XH_B2B-XH-AM_1x02_P2.50mm_Vertical
- J4: value (none) -> DX07S016JA1R1500; footprint (none) -> usbccon:JAE_DX07S016JA1R1500
- J5: value (none) -> Accessory 0; footprint (none) -> Connector_JST:JST_PH_B4B-PH-K_1x04_P2.00mm_Vertical
- J6: value (none) -> Accessory 1; footprint (none) -> Connector_JST:JST_PH_B4B-PH-K_1x04_P2.00mm_Vertical
- J7: footprint (none) -> Connector_JST:JST_PH_B4B-PH-K_1x04_P2.00mm_Vertical
- R1, R12, R4: value (none) -> 2.2; footprint (none) -> Resistor_SMD:R_0402_1005Metric
- R10, R11: value (none) -> 4.7k; footprint (none) -> Resistor_SMD:R_0402_1005Metric
- R13: value (none) -> 47k; footprint (none) -> Resistor_SMD:R_0402_1005Metric
- R14: value (none) -> 470; footprint (none) -> Resistor_SMD:R_0402_1005Metric
- R17, R18, R8, R9: value (none) -> 27; footprint (none) -> Resistor_SMD:R_0402_1005Metric
- R19: value (none) -> 0; footprint (none) -> Resistor_SMD:R_0402_1005Metric
- R2, R3: value (none) -> 0.11; footprint (none) -> Resistor_SMD:R_0805_2012Metric
- R5: value (none) -> 10k; footprint (none) -> Resistor_SMD:R_0402_1005Metric
- R6, R7: value (none) -> 5.1k; footprint (none) -> Resistor_SMD:R_0402_1005Metric
- TH1: value (none) -> Thermistor_NTC; footprint (none) -> Resistor_SMD:R_0402_1005Metric
- U1: value (none) -> HolyIot-18010; footprint (none) -> Phischbol:HOLYIOT-18010
- U2: value (none) -> TMC2130-LA; footprint (none) -> Package_DFN_QFN:QFN-36-1EP_5x6mm_P0.5mm_EP3.6x4.1mm_ThermalVias
- U4: value (none) -> TLV76033DBZT; footprint (none) -> footprints:TLV76033DBZT
Connections:
- net +12V: now also R20.1
- net ACC0_A: now also U1.35 (P0.09); no longer U1.2 (P1.11)
- net ACC0_B: now also U1.36 (P0.10); no longer U1.3 (P1.10)
- net GND: now also C19.2, D3.1 (K), D4.1 (K), R21.2
- net at U1.15 (P0.07): now also R15.2
- net at U1.16 (P1.09): now also R16.2
- new net: D3.2 (A), R15.1
- new net: D4.2 (A), R16.1
- new net Vmeas: C19.1, R20.2, R21.1, U1.3 (P1.10)
Other:
- moved on the sheet: J2, R4, R5
